File: hardware/Kit_Alebrije/Kit_Alebrije.kicad_pcb (KiCad board)
At the start: 2 copper layers, 40.6 x 60 mm, 13 parts, among them Q1 BC547, Q2 BC547, SW2 On

Commit message: feat(Hw):Sw_Updated
unit's_Footprint_Added
Parts:
- SW2: footprint Button_Switch_SMD:SW_SPDT_Shouhan_MSK12C02 -> Kits:SW-SMD_3P-P1.50_L2.7-W6.6
- moved SW2 1.19 mm to (160.0, 59.8)
- moved kibuzzard-6AC559DE 1.14 mm to (156.0, 60.3)
Routing:
- net Net-(BT1--): track 53.3 -> 52.5 mm
