File: hardware/Kit_Esoterico/Kit_Esoterico.kicad_pcb (KiCad board)
At the start: 2 copper layers, 60 x 59 mm, 13 parts, among them Q1 BC547, Q2 BC547, SW2 On

Commit message: feat(Hw):Sw_Updated
unit's_Footprint_Added
Parts:
- SW2: footprint Button_Switch_SMD:SW_SPDT_Shouhan_MSK12C02 -> Kits:SW-SMD_3P-P1.50_L2.7-W6.6
- moved SW2 0.61 mm to (106.9, 53.1)
