File: hardware/Kit_Esoterico/Kit_Esoterico.kicad_sch (KiCad schematic)
At the start: 12 parts, among them Q3 BC548, Q4 BC548, SW2 On

Commit message: feat(Hw):Projects_Added
Parts:
- removed Q3, Q4: BC548, Package_TO_SOT_THT:TO-92_Inline_Horizontal2, symbol Transistor_BJT:BC548
- added Q1, Q2: BC547, Package_TO_SOT_THT:TO-92_Inline_Horizontal1, symbol Transistor_BJT:BC547
Connections:
- net GND: now also Q1.1 (E), Q2.1 (E)
- net at C3.2, R3.2: now also Q2.2 (B)
- net at C4.1, D2.2 (A), R1.2: now also Q2.3 (C)
- net at C4.2, R2.2: now also Q1.2 (B)
- net at C3.1, D1.2 (A), R4.2: now also Q1.3 (C)

Commit message: feat(Hw):Sw_Updated
unit's_Footprint_Added
Parts:
- SW2: footprint Button_Switch_SMD:SW_SPDT_Shouhan_MSK12C02 -> Kits:SW-SMD_3P-P1.50_L2.7-W6.6
Changed lines of the file:
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@@
 			)
 		)
-		(property "Footprint" "Button_Switch_SMD:SW_SPDT_Shouhan_MSK12C02"
+		(property "Footprint" "Kits:SW-SMD_3P-P1.50_L2.7-W6.6"
 			(at 204.47 55.88 0)
 			(hide yes)
