File: hardware/Kit_Mariachi/Kit_Mariachi.kicad_pcb (KiCad board)
At the start: 2 copper layers, 57.3 x 60 mm, 13 parts, among them Q1 BC547, Q2 BC547, SW2 On

Commit message: feat(Hw):Sw_Updated
unit's_Footprint_Added
Parts:
- SW2: footprint Button_Switch_SMD:SW_SPDT_Shouhan_MSK12C02 -> Kits:SW-SMD_3P-P1.50_L2.7-W6.6
- moved SW2 0.75 mm to (186.0, 65.5)
Routing:
- net GND: vias 0 -> 2
