File: hardware/Kit_Robot/Kit_Robot.kicad_sch (KiCad schematic)
At the start: 12 parts, among them Q3 BC548, Q4 BC548, SW2 On

Commit message: feat(Hw):Sw_Updated
unit's_Footprint_Added
Parts:
- SW2: footprint Button_Switch_SMD:SW_SPDT_Shouhan_MSK12C02 -> Kits:SW-SMD_3P-P1.50_L2.7-W6.6
Changed lines of the file:
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@@
 			)
 		)
-		(property "Footprint" "Button_Switch_SMD:SW_SPDT_Shouhan_MSK12C02"
+		(property "Footprint" "Kits:SW-SMD_3P-P1.50_L2.7-W6.6"
 			(at 172.72 86.36 0)
 			(hide yes)
